Commit message: nav2 implemented

File: src/my_scout_description/urdf/scout_mini.xacro (robot description, xacro)
@@ -22,5 +22,5 @@
             <origin xyz="0 0 0" />
             <inertia ixx="0.185196122711036" ixy="4.30144213829512E-08" ixz="5.81037523686401E-08"
-                     iyy="0.364893736238929" iyz="-0.000386720198091934" izz="0.223868521722778" />
+                     iyy="0.273670302179197" iyz="-0.000386720198091934" izz="0.167901391292084" />
         </inertial>
     </link>
@@ -54,6 +54,14 @@
         <parent link="base_link" />
         <child link="front_right_wheel_link" />
-        <axis xyz="0 0 -1" rpy="0 0 0" />
-    </joint>
+        <axis xyz="0 0 -1" />
+    </joint>
+    <!-- Gazebo friction for front right wheel -->
+    <gazebo reference="front_right_wheel_link">
+        <mu1>0.5</mu1>
+        <mu2>0.5</mu2>
+        <kp>1000000.0</kp>
+        <kd>100.0</kd>
+        <minDepth>0.001</minDepth>
+    </gazebo>
     <!-- Front Left Wheel -->
     <link name="front_left_wheel_link">
@@ -80,6 +88,14 @@
         <parent link="base_link" />
         <child link="front_left_wheel_link" />
-        <axis xyz="0 0 1" rpy="0 0 0" />
-    </joint>
+        <axis xyz="0 0 1" />
+    </joint>
+    <!-- Gazebo friction for front left wheel -->
+    <gazebo reference="front_left_wheel_link">
+        <mu1>0.5</mu1>
+        <mu2>0.5</mu2>
+        <kp>1000000.0</kp>
+        <kd>100.0</kd>
+        <minDepth>0.001</minDepth>
+    </gazebo>
     <!-- Rear Right Wheel -->
     <link name="rear_right_wheel_link">
@@ -106,6 +122,14 @@
         <parent link="base_link" />
         <child link="rear_right_wheel_link" />
-        <axis xyz="0 0 -1" rpy="0 0 0" />
-    </joint>
+        <axis xyz="0 0 -1" />
+    </joint>
+    <!-- Gazebo friction for rear right wheel -->
+    <gazebo reference="rear_right_wheel_link">
+        <mu1>0.5</mu1>
+        <mu2>0.5</mu2>
+        <kp>1000000.0</kp>
+        <kd>100.0</kd>
+        <minDepth>0.001</minDepth>
+    </gazebo>
     <!-- Rear Left Wheel -->
     <link name="rear_left_wheel_link">
@@ -132,6 +156,14 @@
         <parent link="base_link" />
         <child link="rear_left_wheel_link" />
-        <axis xyz="0 0 1" rpy="0 0 0" />
-    </joint>
+        <axis xyz="0 0 1" />
+    </joint>
+    <!-- Gazebo friction for rear left wheel -->
+    <gazebo reference="rear_left_wheel_link">
+        <mu1>0.5</mu1>
+        <mu2>0.5</mu2>
+        <kp>1000000.0</kp>
+        <kd>100.0</kd>
+        <minDepth>0.001</minDepth>
+    </gazebo>
     <!-- LiDAR Sensor -->
     <link name="lidar_link">
@@ -163,54 +195,48 @@
         <child link="lidar_link"/>
     </joint>
-      <!-- LiDAR Plugin -->
+    <!-- LiDAR Plugin -->
     <gazebo reference="lidar_link">
-    <sensor name="lidar" type="gpu_lidar">
-    <!-- CHANGED: publish PointCloud2 instead of LaserScan -->
-    <topic>rslidar_points</topic>
-    <ignition_frame_id>lidar_link</ignition_frame_id>
-    <!-- CHANGED: Helios-16P rotates at 10Hz -->
-    <update_rate>10</update_rate>
-    <lidar>
-      <scan>
-        <!-- SAME: 360 horizontal, but denser -->
-        <horizontal>
-          <samples>1800</samples>          <!-- CHANGED: higher resolution -->
-          <resolution>1</resolution>
-          <min_angle>-3.14159</min_angle>
-          <max_angle>3.14159</max_angle>
-        </horizontal>
-        <!-- NEW: 16 vertical beams to simulate RS-Helios -->
-        <vertical>
-          <samples>16</samples>            <!-- NEW -->
-          <resolution>1</resolution>       <!-- NEW -->
-          <min_angle>-0.261799</min_angle> <!-- NEW (−15°) -->
-          <max_angle>0.261799</max_angle>  <!-- NEW (+15°) -->
-        </vertical>
-      </scan>
-      <!-- CHANGED: Range of RS-Helios up to 100 m -->
-      <range>
-        <min>0.2</min>
-        <max>100.0</max>
-        <resolution>0.01</resolution>
-      </range>
-    </lidar>
-    <always_on>1</always_on>
-    <visualize>true</visualize>
-  </sensor>
-</gazebo>
-        <!-- Camera Sensor -->
+        <sensor name="lidar" type="gpu_lidar">
+            <topic>scan</topic>
+            <ignition_frame_id>lidar_link</ignition_frame_id>
+            <update_rate>10</update_rate>
+            <lidar>
+                <scan>
+                    <horizontal>
+                        <samples>360</samples>
+                        <resolution>1</resolution>
+                        <min_angle>-3.14159</min_angle>
+                        <max_angle>3.14159</max_angle>
+                    </horizontal>
+                </scan>
+                <range>
+                    <min>0.12</min>
+                    <max>10.0</max>
+                    <resolution>0.01</resolution>
+                </range>
+                <noise>
+                    <type>gaussian</type>
+                    <mean>0.0</mean>
+                    <stddev>0.01</stddev>
+                </noise>
+            </lidar>
+            <always_on>1</always_on>
+            <visualize>true</visualize>
+        </sensor>
+    </gazebo>
+    <!-- Camera Sensor -->
     <link name="camera_link">
         <inertial>
             <mass value="0.1"/>
             <origin xyz="0 0 0"/>
-            <inertia ixx="0.0001" ixy="0" ixz="0" iyy="0.0001" iyz="0" izz="0.0001"/>
+            <inertia ixx="0.00005" ixy="0" ixz="0" iyy="0.00005" iyz="0" izz="0.00005"/>
         </inertial>
         <visual>
             <origin xyz="0 0 0" rpy="0 0 0"/>
             <geometry>
-                <box size="0.05 0.05 0.05"/>
-            </geometry>
-            <material name="blue">
-                <color rgba="0.0 0.0 0.8 1"/>
+                <box size="0.04 0.08 0.03"/>
+            </geometry>
+            <material name="dark_gray">
+                <color rgba="0.2 0.2 0.2 1"/>
             </material>
         </visual>
@@ -218,5 +244,5 @@
             <origin xyz="0 0 0" rpy="0 0 0"/>
             <geometry>
-                <box size="0.05 0.05 0.05"/>
+                <box size="0.04 0.08 0.03"/>
             </geometry>
         </collision>
@@ -272,11 +298,11 @@
             <left_joint>rear_left_wheel</left_joint>
             <right_joint>rear_right_wheel</right_joint>
-            <wheel_separation>0.58</wheel_separation>
+            <wheel_separation>0.845</wheel_separation>
             <wheel_radius>0.08</wheel_radius>
             <max_wheel_torque>20</max_wheel_torque>
             <max_linear_acceleration>1.0</max_linear_acceleration>
+            <max_angular_acceleration>2.0</max_angular_acceleration>
             <topic>cmd_vel</topic>
             <odom_topic>odom</odom_topic>
-            <tf_topic>tf</tf_topic>
             <odom_publish_frequency>50</odom_publish_frequency>
             <frame_id>odom</frame_id>
